File: business_card_board/business_card_board.kicad_pcb (KiCad board)
At the start: 2 copper layers, 85 x 54 mm, 23 parts, among them J1 PICKit3_Programmer, U1 PIC12F1822

Commit message: v1.1 gerbers finalised
Parts:
- turned -> to 270 degrees
- turned <- to 270 degrees
Routing:
- net VPP/~MCLR: track 84.9 -> 79.8 mm
- net Net-(R1-Pad2): track 92.3 -> 87.3 mm
- net Net-(D1-Pad2): track 40.3 -> 38.1 mm
- net GND: track 71.2 -> 72.1 mm
